File: stm32f072c8_mcu.kicad_pcb (KiCad board)
At the start: 4 copper layers, 70 x 40 mm, 35 parts, among them J1 Conn_01x18_Socket, J2 Conn_01x18_Socket, J3 Conn_01x03_Pin, SW1 SW_Push, U1 STM32F072CBTx, U2 USBLC6-2SC6, U4 AP7384-33SA

Commit message: dasdsad
Parts:
- added C12: 100n, Capacitor_SMD:C_0603_1608Metric, F.Cu at (148.5, 92.0)
- added C13: 100n, Capacitor_SMD:C_0603_1608Metric, F.Cu at (148.6, 103.7)
- added C14: 1u, Capacitor_SMD:C_0603_1608Metric, F.Cu at (166.2, 103.8)
- added C15: 100n, Capacitor_SMD:C_0603_1608Metric, F.Cu at (167.1, 97.0)
- added D2: LED, LED_SMD:LED_PLCC-2_3x2mm_KA, F.Cu at (168.5, 89.0)
- added R10: 10k, Resistor_SMD:R_0603_1608Metric, F.Cu at (166.2, 105.4)
- added R11: 10k, Resistor_SMD:R_0603_1608Metric, F.Cu at (168.5, 104.6)
- added R12: 10k, Resistor_SMD:R_0603_1608Metric, F.Cu at (166.3, 92.9)
- added SW2: SW_Push, Button_Switch_SMD:SW_Push_SPST_NO_Alps_SKRK, F.Cu at (168.5, 109.9)
- added U5: ~, Package_SO:SOIC-16W_7.5x10.3mm_P1.27mm, F.Cu at (155.5, 94.1)
- added U6: ~, Package_SO:SOIC-16W_7.5x10.3mm_P1.27mm, F.Cu at (155.5, 106.1)
- added U7: 74AHC1G14, Package_TO_SOT_SMD:SOT-353_SC-70-5_Handsoldering, F.Cu at (168.5, 100.2)
- C9: value C -> 100n
- R3, R4: value 27 -> 10k
- moved R4 35.2 mm to (162.3, 108.5), turned to -90 degrees
- moved R3 4.62 mm to (147.9, 89.6)
- moved R2 2.08 mm to (135.8, 90.1), turned to -90 degrees
- moved C5 1.31 mm to (126.0, 93.1)
- moved C4 0.31 mm to (126.0, 91.0), turned to 0 degrees
Connections:
- net SPI1_CS_NAND renamed ~{SPI1_NAND_CS}
- net SPI1_CS_NOR renamed ~{SPI1_NOR_CS}
- J1 pad 15: PF0 -> GND
- J1 pad 16: PF1 -> GND
- J2 pad 3: PA10 -> +3.3V
- R3 pad 1: SPI1_MISO -> +3.3V
- R3 pad 2: SPI1_MISO -> ~{SPI1_NAND_HOLD}
- R4 pad 1: SPI1_MOSI -> +3.3V
- R4 pad 2: SPI1_MOSI -> ~{SPI1_NOR_HOLD}
- U1 pad 31: PA10 -> +3.3V
- U1 pad 5: PF0 -> USR_BTN
- U1 pad 6: PF1 -> USR_LED
Routing:
- net USR_BTN: track 0.00 -> 50.2 mm, vias 0 -> 2
- net GND: track 33.9 -> 78.8 mm, vias 23 -> 35
- net +3.3V: track 20.3 -> 58.2 mm, vias 8 -> 16
- net USR_LED: track 0.00 -> 36.7 mm, vias 0 -> 2
- net SPI1_MISO: track 17.8 -> 50.2 mm, vias 0 -> 2
- net SPI1_SCK: track 14.1 -> 46.2 mm, vias 0 -> 2
- net PF1: track 30.5 -> 0.00 mm, vias 1 -> 0
- net PF0: track 27.7 -> 0.00 mm, vias 1 -> 0
- net SPI1_MOSI: track 17.6 -> 42.6 mm, vias 0 -> 4
- net ~{SPI1_NOR_CS}: track 6.91 -> 30.3 mm
- net PA10: track 21.4 -> 0.00 mm
- net ~{SPI1_NOR_HOLD}: track 0.00 -> 20.5 mm
- net ~{SPI1_NAND_HOLD}: track 0.00 -> 17.3 mm
- net ~{SPI1_NAND_CS}: track 8.51 -> 21.3 mm, vias 0 -> 2
- net PB13: track 21.6 -> 18.2 mm, vias 0 -> 1
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- added copper zone on In2.Cu, net +3.3V
- added copper zone on In1.Cu, net GND
- removed copper zone on In1.Cu, net +3.3V
Other:
- board text removed: "PF0"
- board text removed: "PF1"

Commit message: fsdfsdf
Parts:
- removed D2: LED, LED_SMD:LED_PLCC-2_3x2mm_KA
- removed R12: 10k, Resistor_SMD:R_0603_1608Metric
- added D6: LED_RGBA, custom:2.8x3.5_LED_RGB, F.Cu at (158.5, 83.5)
- added J4: Conn_01x14_Socket, Connector_PinSocket_2.54mm:PinSocket_1x14_P2.54mm_Vertical, F.Cu at (113.7, 83.5)
- added R15: 220, Resistor_SMD:R_0603_1608Metric, F.Cu at (159.9, 86.5)
- added R16: 10k, Resistor_SMD:R_0603_1608Metric, F.Cu at (137.3, 108.0)
- added R17: 220, Resistor_SMD:R_0603_1608Metric, F.Cu at (153.7, 84.8)
- added R18: 220, Resistor_SMD:R_0603_1608Metric, F.Cu at (153.7, 82.8)
- J1: value Conn_01x18_Socket -> Conn_01x02_Pin; footprint Connector_PinSocket_2.54mm:PinSocket_1x18_P2.54mm_Vertical -> Connector_PinHeader_2.54mm:PinHeader_1x02_P2.54mm_Vertical
- J2: value Conn_01x18_Socket -> Conn_01x05_Pin; footprint Connector_PinSocket_2.54mm:PinSocket_1x18_P2.54mm_Vertical -> Connector_PinHeader_2.54mm:PinHeader_1x05_P2.54mm_Vertical
- J3: value Conn_01x03_Pin -> Conn_01x14_Socket; footprint Connector_PinHeader_2.54mm:PinHeader_1x03_P2.54mm_Vertical -> Connector_PinSocket_2.54mm:PinSocket_1x14_P2.54mm_Vertical
- moved J2 55.1 mm to (168.5, 89.6), turned to 0 degrees
- moved J1 30.0 mm to (142.7, 108.8), turned to -90 degrees
- moved J3 28.0 mm to (113.7, 116.5)
- moved C15 23.1 mm to (153.9, 115.9), turned to -90 degrees
- moved U7 18.2 mm to (157.2, 114.5), turned to 180 degrees
- moved C14 12.3 mm to (161.8, 115.3), turned to -90 degrees
- moved R10 10.3 mm to (163.5, 115.3), turned to 90 degrees
- moved R11 10.2 mm to (162.6, 113.0), turned to 0 degrees
- moved R1 0.82 mm to (109.2, 114.1), turned to -90 degrees
- moved C4 0.77 mm to (125.2, 90.9)
- moved SW2 0.71 mm to (168.5, 110.6), turned to -90 degrees
- moved C5 0.51 mm to (126.5, 93.1)
- moved C1 0.45 mm to (138.5, 97.2)
Connections:
- J1 pad 2: PA13 -> BOOT0
- J2 pad 2: +5V_VBUS -> SWDIO
- J2 pad 3: +3.3V -> SWCLK
- J2 pad 4: PA9 -> NRST
- J2 pad 5: PA8 -> GND
- J3 pad 2: BOOT0 -> PA10
- J3 pad 3: GND -> PA15
- R1 pad 2: NRST -> +3.3V
- U1 pad 10: PA0 -> USR_LED_R
- U1 pad 11: PA1 -> USR_LED_G
- U1 pad 12: PA2 -> USR_LED_B
- U1 pad 31: +3.3V -> PA10
- U1 pad 34: PA13 -> SWDIO
- U1 pad 37: PA14 -> SWCLK
- U1 pad 4: PC15 -> USR_BTN
- U1 pad 5: USR_BTN -> OSC_IN
- U1 pad 6: USR_LED -> OSC_OUT
Routing:
- net SWDIO: track 0.00 -> 44.9 mm, vias 0 -> 1
- net SWCLK: track 0.00 -> 44.0 mm, vias 0 -> 1
- net NRST: track 35.0 -> 73.1 mm, vias 0 -> 3
- net USR_LED: track 36.7 -> 0.00 mm, vias 2 -> 0
- net USR_LED_R: track 0.00 -> 32.5 mm, vias 0 -> 2
- net PA10: track 0.00 -> 28.3 mm
- net USR_LED_G: track 0.00 -> 26.3 mm, vias 0 -> 2
- net USR_LED_B: track 0.00 -> 25.8 mm, vias 0 -> 2
- net PA0: track 25.0 -> 0.00 mm, vias 1 -> 0
- net PC15: track 24.0 -> 0.00 mm, vias 1 -> 0
- net PA1: track 22.5 -> 0.00 mm, vias 1 -> 0
- net PA13: track 22.3 -> 0.00 mm, vias 1 -> 0
- net PA2: track 19.7 -> 0.00 mm, vias 1 -> 0
- net PA14: track 18.8 -> 0.00 mm, vias 1 -> 0
- net +3.3V: track 58.2 -> 41.2 mm, vias 16 -> 21
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Other:
- board text added: "NRST"
- board text added: "SWCLK"
- board text added: "SWIO"
- board text removed: "BOOT0"
- board text removed: "PA0"
- board text removed: "PA1"
- board text removed: "PA13"
- board text removed: "PA14"
- board text removed: "PA2"
- board text removed: "PC15"

Commit message: sdsdfsd
Parts:
- removed D6: LED_RGBA, custom:2.8x3.5_LED_RGB
- added C12: 22p, Capacitor_SMD:C_0603_1608Metric, F.Cu at (140.7, 107.1)
- added C13: 22p, Capacitor_SMD:C_0603_1608Metric, F.Cu at (143.9, 101.9)
- added D2: LED, LED_SMD:LED_PLCC-2_3x2mm_KA, F.Cu at (105.5, 89.9)
- added Y1: 16MHz, custom:3225_smd_crystal, F.Cu at (143.1, 105.2)
- D1: value LED -> APFA3010; footprint LED_SMD:LED_PLCC-2_3x2mm_KA -> custom:2.8x3.5_LED_RGB
- moved D1 54.1 mm to (159.2, 83.5), turned to 180 degrees
- moved J1 14.4 mm to (128.3, 110.0), turned to 90 degrees
- moved R9 9.94 mm to (163.6, 86.5), turned to 90 degrees
- moved R8 6.38 mm to (153.7, 84.8), turned to 180 degrees
- moved R3 3.45 mm to (134.6, 110.0), turned to 180 degrees
- moved G*** 1.08 mm to (119.9, 107.5)
- moved R11 0.87 mm to (111.7, 105.9)
- moved R12 0.21 mm to (112.7, 95.0)
- renumbered C14 to C10, C9 to C11, C10 to C14, C11 to C15, C13 to C16, C12 to C17, C15 to C9, R10 to R1, R18 to R10, R7 to R11, R8 to R12, R9 to R13, R3 to R14, R4 to R15, R11 to R2, R16 to R3, R1 to R4, R2 to R5, R5 to R6, R6 to R7, R15 to R8, R17 to R9, SW2 to SW1, SW1 to SW2, U7 to U1, U1 to U2, U2 to U3, U3 to U4, U4 to U5, U5 to U6, U6 to U7
Connections:
- D1 pad 1: /USB/PWR_LED -> USR_LED_R
- U2 pad 10: USR_LED_R -> USR_LED_G
- U2 pad 11: USR_LED_G -> USR_LED_R
Routing:
- net OSC_IN: track 0.00 -> 13.7 mm
- net OSC_OUT: track 0.00 -> 11.3 mm
- net USR_LED_G: track 26.3 -> 36.9 mm
- net GND: track 82.7 -> 90.0 mm, vias 44 -> 51
- net USR_LED_R: track 32.5 -> 25.8 mm
- net +3.3V: track 41.2 -> 38.7 mm, vias 21 -> 20
- net +5V_VBUS: track 29.8 -> 32.2 mm, vias 3 -> 2
- net BOOT0: track 12.1 -> 10.4 mm
- net PB7: track 14.0 -> 15.2 mm
- net PB6: track 14.2 -> 15.3 mm
- net USR_LED_B: track 25.8 -> 25.3 mm
