File: sheets/flash.kicad_sch (KiCad schematic)
At the start: 0 parts

Commit message: dasdsad
Parts:
- added C12, C13: 100n, Capacitor_SMD:C_0603_1608Metric, symbol Device:C
- added R3, R4: 10k, Resistor_SMD:R_0603_1608Metric, symbol Device:R
- added U5: ~, Package_SO:SOIC-16W_7.5x10.3mm_P1.27mm, symbol custom:W25N512GVFIR
- added U6: ~, Package_SO:SOIC-16W_7.5x10.3mm_P1.27mm, symbol custom:W25Q64JVSFIM
Connections:
- new net +3.3V: C12.1, C13.1, R3.1, R4.1, U5.2 (VCC), U6.2 (VCC)
- new net GND: C12.2, C13.2, U5.10 (GND), U5.11 (N/C), U5.12 (N/C), U5.13 (N/C), U5.14 (N/C), U5.3 (N/C), U5.4 (N/C), U5.5 (N/C), U5.6 (N/C), U6.10 (GND), U6.11 (N/C), U6.12 (N/C), U6.13 (N/C), U6.14 (N/C), U6.4 (N/C), U6.5 (N/C), U6.6 (N/C)
- new net SPI1_MISO: U5.15 (DI(IO_{0})), U6.15 (DI(IO_{0}))
- new net SPI1_MOSI: U5.8 (DO(IO_{1})), U6.8 (DO(IO_{1}))
- new net SPI1_SCK: U5.16 (CLK), U6.16 (CLK)
- new net ~{SPI1_NAND_CS}: U5.7 (~{CS})
- new net ~{SPI1_NAND_HOLD}: R3.2, U5.1 (~{HOLD}(IO_{3})), U5.9 (~{WP}(IO_{2}))
- new net ~{SPI1_NOR_CS}: U6.7 (~{CS})
- new net ~{SPI1_NOR_HOLD}: R4.2, U6.1 (~{HOLD}(IO_{3})), U6.3 (~{RESET}), U6.9 (~{WP}(IO_{2}))

Commit message: sdsdfsd
Parts:
- renumbered C13 to C16, C12 to C17, R3 to R14, R4 to R15, U5 to U6, U6 to U7
Changed lines of the file:
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@@
 		(dnp no)
 		(fields_autoplaced yes)
-		(property "Reference" "U5"
+		(property "Reference" "U6"
 			(at 226.9841 34.29 0)
 			(effects
@@
 			(project ""
 				(path "/e68034de-3c5e-4df9-b3d4-7e0ea1d00387/35d32fe6-594a-4259-8115-e203447d539d"
-					(reference "U5")
+					(reference "U6")
 					(unit 1)
 				)
@@
 		(dnp no)
 		(fields_autoplaced yes)
-		(property "Reference" "#PWR033"
+		(property "Reference" "#PWR050"
 			(at 224.79 133.35 0)
 			(effects
@@
 			(project ""
 				(path "/e68034de-3c5e-4df9-b3d4-7e0ea1d00387/35d32fe6-594a-4259-8115-e203447d539d"
-					(reference "#PWR033")
+					(reference "#PWR050")
 					(unit 1)
 				)
@@
 		(dnp no)
 		(fields_autoplaced yes)
-		(property "Reference" "#PWR037"
+		(property "Reference" "#PWR044"
 			(at 92.71 48.26 0)
 			(effects
@@
 			(project "stm32f072c8_mcu"
 				(path "/e68034de-3c5e-4df9-b3d4-7e0ea1d00387/35d32fe6-594a-4259-8115-e203447d539d"
-					(reference "#PWR037")
+					(reference "#PWR044")
 					(unit 1)
 				)
@@
 		(dnp no)
 		(fields_autoplaced yes)
-		(property "Reference" "#PWR039"
+		(property "Reference" "#PWR048"
 			(at 50.8 83.82 0)
 			(effects
@@
 			(project "stm32f072c8_mcu"
 				(path "/e68034de-3c5e-4df9-b3d4-7e0ea1d00387/35d32fe6-594a-4259-8115-e203447d539d"
-					(reference "#PWR039")
+					(reference "#PWR048")
 					(unit 1)
 				)
@@
 		(dnp no)
 		(fields_autoplaced yes)
-		(property "Reference" "U6"
+		(property "Reference" "U7"
 			(at 226.9841 93.98 0)
 			(effects
@@
 			(project ""
 				(path "/e68034de-3c5e-4df9-b3d4-7e0ea1d00387/35d32fe6-594a-4259-8115-e203447d539d"
-					(reference "U6")
+					(reference "U7")
 					(unit 1)
 				)
@@
 		(dnp no)
 		(fields_autoplaced yes)
-		(property "Reference" "#PWR036"
+		(property "Reference" "#PWR042"
 			(at 92.71 33.02 0)
 			(effects
@@
 			(project "stm32f072c8_mcu"
 				(path "/e68034de-3c5e-4df9-b3d4-7e0ea1d00387/35d32fe6-594a-4259-8115-e203447d539d"
-					(reference "#PWR036")
+					(reference "#PWR042")
 					(unit 1)
 				)
@@
 		(dnp no)
 		(fields_autoplaced yes)
-		(property "Reference" "C12"
+		(property "Reference" "C17"
 			(at 107.95 34.2899 0)
 			(effects
@@
 			(project ""
 				(path "/e68034de-3c5e-4df9-b3d4-7e0ea1d00387/35d32fe6-594a-4259-8115-e203447d539d"
-					(reference "C12")
+					(reference "C17")
 					(unit 1)
 				)
@@
 		(dnp no)
 		(fields_autoplaced yes)
-		(property "Reference" "#PWR031"
+		(property "Reference" "#PWR049"
 			(at 224.79 97.79 0)
 			(effects
@@
 			(project "stm32f072c8_mcu"
 				(path "/e68034de-3c5e-4df9-b3d4-7e0ea1d00387/35d32fe6-594a-4259-8115-e203447d539d"
-					(reference "#PWR031")
+					(reference "#PWR049")
 					(unit 1)
 				)
@@
 		(dnp no)
 		(fields_autoplaced yes)
-		(property "Reference" "#PWR035"
+		(property "Reference" "#PWR051"
 			(at 242.57 133.35 0)
 			(effects
@@
 			(project "stm32f072c8_mcu"
 				(path "/e68034de-3c5e-4df9-b3d4-7e0ea1d00387/35d32fe6-594a-4259-8115-e203447d539d"
-					(reference "#PWR035")
+					(reference "#PWR051")
 					(unit 1)
 				)
@@
 		(on_board yes)
 		(dnp no)
-		(property "Reference" "R4"
+		(property "Reference" "R15"
 			(at 51.816 85.09 0)
 			(effects
@@
 			(project "stm32f072c8_mcu"
 				(path "/e68034de-3c5e-4df9-b3d4-7e0ea1d00387/35d32fe6-594a-4259-8115-e203447d539d"
-					(reference "R4")
+					(reference "R15")
 					(unit 1)
 				)
@@
 		(dnp no)
 		(fields_autoplaced yes)
-		(property "Reference" "C13"
+		(property "Reference" "C16"
 			(at 96.52 34.2899 0)
 			(effects
@@
 			(project "stm32f072c8_mcu"
 				(path "/e68034de-3c5e-4df9-b3d4-7e0ea1d00387/35d32fe6-594a-4259-8115-e203447d539d"
-					(reference "C13")
+					(reference "C16")
 					(unit 1)
 				)
@@
 		(dnp no)
 		(fields_autoplaced yes)
-		(property "Reference" "#PWR034"
+		(property "Reference" "#PWR047"
 			(at 242.57 73.66 0)
 			(effects
@@
 			(project "stm32f072c8_mcu"
 				(path "/e68034de-3c5e-4df9-b3d4-7e0ea1d00387/35d32fe6-594a-4259-8115-e203447d539d"
-					(reference "#PWR034")
+					(reference "#PWR047")
 					(unit 1)
 				)
@@
 		(on_board yes)
 		(dnp no)
-		(property "Reference" "R3"
+		(property "Reference" "R14"
 			(at 51.816 58.42 0)
 			(effects
@@
 			(project ""
 				(path "/e68034de-3c5e-4df9-b3d4-7e0ea1d00387/35d32fe6-594a-4259-8115-e203447d539d"
-					(reference "R3")
+					(reference "R14")
 					(unit 1)
 				)
@@
 		(dnp no)
 		(fields_autoplaced yes)
-		(property "Reference" "#PWR038"
+		(property "Reference" "#PWR045"
 			(at 50.8 57.15 0)
 			(effects
@@
 			(project "stm32f072c8_mcu"
 				(path "/e68034de-3c5e-4df9-b3d4-7e0ea1d00387/35d32fe6-594a-4259-8115-e203447d539d"
-					(reference "#PWR038")
+					(reference "#PWR045")
 					(unit 1)
 				)
@@
 		(dnp no)
 		(fields_autoplaced yes)
-		(property "Reference" "#PWR032"
+		(property "Reference" "#PWR046"
 			(at 224.79 73.66 0)
 			(effects
@@
 			(project ""
 				(path "/e68034de-3c5e-4df9-b3d4-7e0ea1d00387/35d32fe6-594a-4259-8115-e203447d539d"
-					(reference "#PWR032")
+					(reference "#PWR046")
 					(unit 1)
 				)
@@
 		(dnp no)
 		(fields_autoplaced yes)
-		(property "Reference" "#PWR030"
+		(property "Reference" "#PWR043"
 			(at 224.79 38.1 0)
 			(effects
@@
 			(project ""
 				(path "/e68034de-3c5e-4df9-b3d4-7e0ea1d00387/35d32fe6-594a-4259-8115-e203447d539d"
-					(reference "#PWR030")
-					(unit 1)
-				)
+					(reference "#PWR043")
+					(unit 1)
+				)
