File: sheets/usb.kicad_sch (KiCad schematic)
At the start: 8 parts, among them U3 USBLC6-2SC6, U4 AP7384-33SA

Commit message: fsdfsdf
Parts:
- removed C9: 100n, Capacitor_SMD:C_0603_1608Metric, symbol Device:C
- added D1: LED, LED_SMD:LED_PLCC-2_3x2mm_KA, symbol Device:LED
- added R9: 50, Resistor_SMD:R_0603_1608Metric, symbol Device:R
- renumbered R1 to R7, R2 to R8, U3 to U2, U2 to U3
Connections:
- net 5V VBUS is gone; now on net +5V_VBUS: C10.1, U3.A4 (VBUS), U3.A9 (VBUS), U3.B4 (VBUS), U3.B9 (VBUS), U4.1 (VI)
- net +3.3V: now also D1.2 (A)
- net GND: now also U4.3 (GND), R9.2
- net USB_D+: now also U2.1 (I/O1), U2.6 (I/O1); no longer U2.3 (I/O2), U2.4 (I/O2)
- net USB_D-: now also U2.3 (I/O2), U2.4 (I/O2); no longer U2.1 (I/O1), U2.6 (I/O1)
- net CC1: now reaches R8.1, U3.A5 (CC1)
- net CC2: now reaches R7.1, U3.B5 (CC2)
- net +5V_VBUS: now reaches U2.5 (VBUS)
- new net PWR_LED: D1.1 (K), R9.1
- no-connect marks 0 -> 2

Commit message: dasdsad
Other:
- moved on the sheet: C10, C11, D1, R9, U2, U4

Commit message: sdsdfsd
Parts:
- renumbered C10 to C14, C11 to C15, D1 to D2, R7 to R11, R8 to R12, R9 to R13, U2 to U3, U3 to U4, U4 to U5
Changed lines of the file:
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@@
 		(dnp no)
 		(fields_autoplaced yes)
-		(property "Reference" "#PWR026"
+		(property "Reference" "#PWR036"
 			(at 82.55 96.52 0)
 			(effects
@@
 			(project "stm32f072c8_mcu"
 				(path "/e68034de-3c5e-4df9-b3d4-7e0ea1d00387/d33bead4-075b-4ab7-8a51-fe807e9b64e0"
-					(reference "#PWR026")
+					(reference "#PWR036")
 					(unit 1)
 				)
@@
 		(on_board yes)
 		(dnp no)
-		(property "Reference" "R8"
+		(property "Reference" "R12"
 			(at 64.516 81.28 0)
 			(effects
@@
 			(project "stm32f072c8_mcu"
 				(path "/e68034de-3c5e-4df9-b3d4-7e0ea1d00387/d33bead4-075b-4ab7-8a51-fe807e9b64e0"
-					(reference "R8")
+					(reference "R12")
 					(unit 1)
 				)
@@
 		(dnp no)
 		(fields_autoplaced yes)
-		(property "Reference" "#PWR021"
+		(property "Reference" "#PWR033"
 			(at 97.79 63.5 0)
 			(effects
@@
 			(project "stm32f072c8_mcu"
 				(path "/e68034de-3c5e-4df9-b3d4-7e0ea1d00387/d33bead4-075b-4ab7-8a51-fe807e9b64e0"
-					(reference "#PWR021")
+					(reference "#PWR033")
 					(unit 1)
 				)
@@
 		(dnp no)
 		(fields_autoplaced yes)
-		(property "Reference" "#PWR023"
+		(property "Reference" "#PWR035"
 			(at 116.84 82.55 0)
 			(effects
@@
 			(project "stm32f072c8_mcu"
 				(path "/e68034de-3c5e-4df9-b3d4-7e0ea1d00387/d33bead4-075b-4ab7-8a51-fe807e9b64e0"
-					(reference "#PWR023")
+					(reference "#PWR035")
 					(unit 1)
 				)
@@
 		(dnp no)
 		(fields_autoplaced yes)
-		(property "Reference" "#PWR025"
+		(property "Reference" "#PWR040"
 			(at 57.15 97.79 0)
 			(effects
@@
 			(project "stm32f072c8_mcu"
 				(path "/e68034de-3c5e-4df9-b3d4-7e0ea1d00387/d33bead4-075b-4ab7-8a51-fe807e9b64e0"
-					(reference "#PWR025")
+					(reference "#PWR040")
 					(unit 1)
 				)
@@
 		(on_board yes)
 		(dnp no)
-		(property "Reference" "#PWR022"
+		(property "Reference" "#PWR034"
 			(at 82.55 82.55 0)
 			(effects
@@
 			(project "stm32f072c8_mcu"
 				(path "/e68034de-3c5e-4df9-b3d4-7e0ea1d00387/d33bead4-075b-4ab7-8a51-fe807e9b64e0"
-					(reference "#PWR022")
+					(reference "#PWR034")
 					(unit 1)
 				)
@@
 		(on_board yes)
 		(dnp no)
-		(property "Reference" "#PWR019"
+		(property "Reference" "#PWR031"
 			(at 57.15 34.29 0)
 			(effects
@@
 			(project ""
 				(path "/e68034de-3c5e-4df9-b3d4-7e0ea1d00387/d33bead4-075b-4ab7-8a51-fe807e9b64e0"
-					(reference "#PWR019")
+					(reference "#PWR031")
 					(unit 1)
 				)
@@
 		(dnp no)
 		(fields_autoplaced yes)
-		(property "Reference" "#PWR027"
+		(property "Reference" "#PWR037"
 			(at 99.06 96.52 0)
 			(effects
@@
 			(project "stm32f072c8_mcu"
 				(path "/e68034de-3c5e-4df9-b3d4-7e0ea1d00387/d33bead4-075b-4ab7-8a51-fe807e9b64e0"
-					(reference "#PWR027")
+					(reference "#PWR037")
 					(unit 1)
 				)
@@
 		(dnp no)
 		(fields_autoplaced yes)
-		(property "Reference" "R9"
+		(property "Reference" "R13"
 			(at 130.81 93.9799 0)
 			(effects
@@
 			(project ""
 				(path "/e68034de-3c5e-4df9-b3d4-7e0ea1d00387/d33bead4-075b-4ab7-8a51-fe807e9b64e0"
-					(reference "R9")
+					(reference "R13")
 					(unit 1)
 				)
@@
 		(dnp no)
 		(fields_autoplaced yes)
-		(property "Reference" "#PWR029"
+		(property "Reference" "#PWR041"
 			(at 128.27 106.68 0)
 			(effects
@@
 			(project "stm32f072c8_mcu"
 				(path "/e68034de-3c5e-4df9-b3d4-7e0ea1d00387/d33bead4-075b-4ab7-8a51-fe807e9b64e0"
-					(reference "#PWR029")
+					(reference "#PWR041")
 					(unit 1)
 				)
@@
 		(on_board yes)
 		(dnp no)
-		(property "Reference" "C11"
+		(property "Reference" "C15"
 			(at 113.03 83.8199 0)
 			(effects
@@
 			(project "stm32f072c8_mcu"
 				(path "/e68034de-3c5e-4df9-b3d4-7e0ea1d00387/d33bead4-075b-4ab7-8a51-fe807e9b64e0"
-					(reference "C11")
+					(reference "C15")
 					(unit 1)
 				)
@@
 		(dnp no)
 		(fields_autoplaced yes)
-		(property "Reference" "#PWR028"
+		(property "Reference" "#PWR038"
 			(at 116.84 96.52 0)
 			(effects
@@
 			(project "stm32f072c8_mcu"
 				(path "/e68034de-3c5e-4df9-b3d4-7e0ea1d00387/d33bead4-075b-4ab7-8a51-fe807e9b64e0"
-					(reference "#PWR028")
+					(reference "#PWR038")
 					(unit 1)
 				)
@@
 		(on_board yes)
 		(dnp no)
-		(property "Reference" "U3"
+		(property "Reference" "U4"
 			(at 33.274 27.94 0)
 			(effects
@@
 			(project ""
 				(path "/e68034de-3c5e-4df9-b3d4-7e0ea1d00387/d33bead4-075b-4ab7-8a51-fe807e9b64e0"
-					(reference "U3")
+					(reference "U4")
 					(unit 1)
 				)
@@
 		(dnp no)
 		(fields_autoplaced yes)
-		(property "Reference" "U2"
+		(property "Reference" "U3"
 			(at 99.4411 38.1 0)
 			(effects
@@
 			(project ""
 				(path "/e68034de-3c5e-4df9-b3d4-7e0ea1d00387/d33bead4-075b-4ab7-8a51-fe807e9b64e0"
-					(reference "U2")
+					(reference "U3")
 					(unit 1)
 				)
@@
 		(dnp no)
 		(fields_autoplaced yes)
-		(property "Reference" "U4"
+		(property "Reference" "U5"
 			(at 99.06 73.66 0)
 			(effects
@@
 			(project ""
 				(path "/e68034de-3c5e-4df9-b3d4-7e0ea1d00387/d33bead4-075b-4ab7-8a51-fe807e9b64e0"
-					(reference "U4")
+					(reference "U5")
 					(unit 1)
 				)
@@
 		(on_board yes)
 		(dnp no)
-		(property "Reference" "C10"
+		(property "Reference" "C14"
 			(at 78.74 83.8199 0)
 			(effects
@@
 			(project "stm32f072c8_mcu"
 				(path "/e68034de-3c5e-4df9-b3d4-7e0ea1d00387/d33bead4-075b-4ab7-8a51-fe807e9b64e0"
-					(reference "C10")
+					(reference "C14")
 					(unit 1)
 				)
@@
 		(dnp no)
 		(fields_autoplaced yes)
-		(property "Reference" "D1"
+		(property "Reference" "D2"
 			(at 132.08 85.4074 90)
 			(effects
@@
 			(project ""
 				(path "/e68034de-3c5e-4df9-b3d4-7e0ea1d00387/d33bead4-075b-4ab7-8a51-fe807e9b64e0"
-					(reference "D1")
+					(reference "D2")
 					(unit 1)
 				)
@@
 		(on_board yes)
 		(dnp no)
-		(property "Reference" "#PWR020"
+		(property "Reference" "#PWR032"
 			(at 97.79 40.64 0)
 			(effects
@@
 			(project "stm32f072c8_mcu"
 				(path "/e68034de-3c5e-4df9-b3d4-7e0ea1d00387/d33bead4-075b-4ab7-8a51-fe807e9b64e0"
-					(reference "#PWR020")
+					(reference "#PWR032")
 					(unit 1)
 				)
@@
 		(on_board yes)
 		(dnp no)
-		(property "Reference" "R7"
+		(property "Reference" "R11"
 			(at 58.166 81.28 0)
 			(effects
@@
 			(project ""
 				(path "/e68034de-3c5e-4df9-b3d4-7e0ea1d00387/d33bead4-075b-4ab7-8a51-fe807e9b64e0"
-					(reference "R7")
+					(reference "R11")
 					(unit 1)
 				)
@@
 		(dnp no)
 		(fields_autoplaced yes)
-		(property "Reference" "#PWR024"
+		(property "Reference" "#PWR039"
 			(at 46.99 97.79 0)
 			(effects
@@
 			(project ""
 				(path "/e68034de-3c5e-4df9-b3d4-7e0ea1d00387/d33bead4-075b-4ab7-8a51-fe807e9b64e0"
-					(reference "#PWR024")
-					(unit 1)
-				)
+					(reference "#PWR039")
+					(unit 1)
+				)
